File: musicman_2EQ.sch (KiCad schematic (older format))
At the start: 27 parts, among them P1 in, P2 rv1.1, P3 rv1.2, P4 rv1.3, P5 rv2.3, P6 rv2.2, P7 out, P8 +9V, P9 Gnd, U1 LM4250

Commit message: board routed
Parts:
- P1, P2, P3, P4, P5, P6, P7, P8, P9: footprint (none) -> Wire_Pads:SolderWirePad_single_0-8mmDrill
Other:
- note added: "Bass"
- note added: "Treble"
Changed lines of the file:
@@
 EESchema Schematic File Version 2
-LIBS:USER
-LIBS:texas_other
 LIBS:power
 LIBS:device
@@
 LIBS:texas
 LIBS:audio
-EELAYER 24 0
+LIBS:USER
+LIBS:texas_other
+LIBS:musicman_2EQ-cache
+EELAYER 25 0
 EELAYER END
 $Descr A4 11693 8268
@@
 F 0 "P2" H 4700 5250 50  0000 C CNN
 F 1 "rv1.1" V 4800 5150 50  0000 C CNN
-F 2 "" H 4700 5150 60  0001 C CNN
+F 2 "Wire_Pads:SolderWirePad_single_0-8mmDrill" H 4700 5150 60  0001 C CNN
 F 3 "" H 4700 5150 60  0000 C CNN
 	1    4700 5150
@@
 F 0 "P3" H 4950 5250 50  0000 C CNN
 F 1 "rv1.2" V 5050 5150 50  0000 C CNN
-F 2 "" H 4950 5150 60  0001 C CNN
+F 2 "Wire_Pads:SolderWirePad_single_0-8mmDrill" H 4950 5150 60  0001 C CNN
 F 3 "" H 4950 5150 60  0000 C CNN
 	1    4950 5150
@@
 F 0 "P4" H 5200 5250 50  0000 C CNN
 F 1 "rv1.3" V 5300 5150 50  0000 C CNN
-F 2 "" H 5200 5150 60  0001 C CNN
+F 2 "Wire_Pads:SolderWirePad_single_0-8mmDrill" H 5200 5150 60  0001 C CNN
 F 3 "" H 5200 5150 60  0000 C CNN
 	1    5200 5150
@@
 F 0 "P7" H 7050 3700 50  0000 C CNN
 F 1 "out" V 7150 3600 50  0000 C CNN
-F 2 "" H 7050 3600 60  0001 C CNN
+F 2 "Wire_Pads:SolderWirePad_single_0-8mmDrill" H 7050 3600 60  0001 C CNN
 F 3 "" H 7050 3600 60  0000 C CNN
 	1    7050 3600
@@
 F 0 "P5" H 7000 2650 50  0000 C CNN
 F 1 "rv2.3" V 7100 2550 50  0000 C CNN
-F 2 "" H 7000 2550 60  0001 C CNN
+F 2 "Wire_Pads:SolderWirePad_single_0-8mmDrill" H 7000 2550 60  0001 C CNN
 F 3 "" H 7000 2550 60  0000 C CNN
 	1    7000 2550
@@
 F 0 "P6" H 7000 2900 50  0000 C CNN
 F 1 "rv2.2" V 7100 2800 50  0000 C CNN
-F 2 "" H 7000 2800 60  0001 C CNN
+F 2 "Wire_Pads:SolderWirePad_single_0-8mmDrill" H 7000 2800 60  0001 C CNN
 F 3 "" H 7000 2800 60  0000 C CNN
 	1    7000 2800
@@
 F 0 "P1" H 3400 3800 50  0000 C CNN
 F 1 "in" V 3500 3700 50  0000 C CNN
-F 2 "" H 3400 3700 60  0001 C CNN
+F 2 "Wire_Pads:SolderWirePad_single_0-8mmDrill" H 3400 3700 60  0001 C CNN
 F 3 "" H 3400 3700 60  0000 C CNN
 	1    3400 3700
@@
 F 0 "P8" H 7750 4050 50  0000 C CNN
 F 1 "+9V" V 7850 3950 50  0000 C CNN
-F 2 "" H 7750 3950 60  0001 C CNN
+F 2 "Wire_Pads:SolderWirePad_single_0-8mmDrill" H 7750 3950 60  0001 C CNN
 F 3 "" H 7750 3950 60  0000 C CNN
 	1    7750 3950
@@
 F 0 "P9" H 7750 5250 50  0000 C CNN
 F 1 "Gnd" V 7850 5150 50  0000 C CNN
-F 2 "" H 7750 5150 60  0001 C CNN
+F 2 "Wire_Pads:SolderWirePad_single_0-8mmDrill" H 7750 5150 60  0001 C CNN
 F 3 "" H 7750 5150 60  0000 C CNN
 	1    7750 5150
@@
 NoConn ~ 7300 2800
 NoConn ~ 5700 3250
+Text Notes 5100 5700 0    60   ~ 0
+Treble
+Text Notes 7700 3000 0    60   ~ 0
+Bass
 $EndSCHEMATC
