File: src/kicad/musicman_2EQ.kicad_pcb (KiCad board)
At the start: 2 copper layers, 44.5 x 21 mm, 25 parts, among them P1 in, P2 rv1.1, P3 rv1.2, P4 rv1.3, P5 rv2.3, P6 rv2.2, P7 out, P8 +9V, P9 Gnd, U1 LM4250

Commit message: 01/11/2014 minor changes
Parts:
- moved P8 0.63 mm to (148.0, 45.1)
Routing:
- net +9V: track 20.3 -> 21.2 mm
Changed lines of the file:
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@@
-(kicad_pcb (version 4) (host pcbnew "(2014-09-19 BZR 5142)-product")
+(kicad_pcb (version 4) (host pcbnew "(2014-10-31 BZR 5247)-product")
   (general
     (links 32)
     (no_connects 0)
-    (area 124.409999 41.148 168.960001 66.429128)
+    (area 124.409999 40.513 168.960001 66.429128)
     (thickness 1.6)
     (drawings 22)
@@
     (visible_elements 7FFEFF7F)
     (pcbplotparams
-      (layerselection 0x010f0_80000001)
-      (usegerberextensions true)
-      (excludeedgelayer true)
+      (layerselection 0x00020_00000000)
+      (usegerberextensions false)
+      (excludeedgelayer false)
       (linewidth 0.100000)
       (plotframeref false)
@@
       (plotvalue false)
       (plotinvisibletext false)
-      (padsonsilk false)
-      (subtractmaskfromsilk true)
-      (outputformat 1)
+      (padsonsilk true)
+      (subtractmaskfromsilk false)
+      (outputformat 4)
       (mirror false)
-      (drillshape 0)
+      (drillshape 2)
       (scaleselection 1)
-      (outputdirectory plots))
+      (outputdirectory ""))
   )
   (net 0 "")
@@
   )
   (module Wire_Pads:SolderWirePad_single_0-8mmDrill (layer F.Cu)
-    (at 147.955 45.72)
+    (at 147.955 45.085)
     (fp_text reference P8 (at 0 -2.54) (layer F.SilkS) hide
       (effects (font (thickness 0.3048)))
@@
   (segment (start 151.13 59.69) (end 153.67 62.23) (width 0.508) (layer B.Cu) (net 6))
   (segment (start 148.59 59.69) (end 151.13 59.69) (width 0.508) (layer B.Cu) (net 6))
-  (segment (start 152.4 45.72) (end 147.955 45.72) (width 0.508) (layer B.Cu) (net 7) (status 20))
-  (segment (start 153.67 46.99) (end 152.4 45.72) (width 0.508) (layer B.Cu) (net 7))
+  (segment (start 149.86 50.8) (end 147.955 48.895) (width 0.508) (layer B.Cu) (net 7))
+  (segment (start 147.955 48.895) (end 147.955 48.26) (width 0.508) (layer B.Cu) (net 7))
+  (segment (start 147.955 48.26) (end 147.955 45.085) (width 0.508) (layer B.Cu) (net 7) (status 20))
+  (segment (start 151.13 50.8) (end 149.86 50.8) (width 0.508) (layer B.Cu) (net 7))
   (segment (start 154.94 45.72) (end 160.02 45.72) (width 0.508) (layer B.Cu) (net 7))
   (segment (start 153.67 46.99) (end 154.94 45.72) (width 0.508) (layer B.Cu) (net 7))
-  (segment (start 147.955 48.26) (end 147.955 45.72) (width 0.508) (layer B.Cu) (net 7))
-  (segment (start 147.955 48.895) (end 147.955 48.26) (width 0.508) (layer B.Cu) (net 7))
-  (segment (start 149.86 50.8) (end 147.955 48.895) (width 0.508) (layer B.Cu) (net 7))
-  (segment (start 151.13 50.8) (end 149.86 50.8) (width 0.508) (layer B.Cu) (net 7))
+  (segment (start 151.765 45.085) (end 147.955 45.085) (width 0.508) (layer B.Cu) (net 7))
+  (segment (start 153.67 46.99) (end 151.765 45.085) (width 0.508) (layer B.Cu) (net 7))
   (segment (start 130.175 62.865) (end 141.605 62.865) (width 0.508) (layer B.Cu) (net 8))
   (segment (start 141.605 62.865) (end 143.51 60.96) (width 0.508) (layer B.Cu) (net 8))
